Commit message: fixed position offset, urdf units

File: gm6020_example/urdf/gm6020.urdf.xacro (robot description, xacro)
@@ -5,5 +5,5 @@
 https://github.com/ros-simulation/gazebo_ros_demos/blob/kinetic-devel/gm6020_description/urdf/gm6020.xacro
 -->
-<robot xmlns:xacro="http://www.ros.org/wiki/xacro" name="2dof_robot">
+<robot xmlns:xacro="http://www.ros.org/wiki/xacro" name="gm6020">
   <xacro:arg name="prefix" default="" />
   <!-- Import Gm6020 macro -->

File: gm6020_example/urdf/gm6020_description.urdf.xacro (robot description, xacro)
@@ -4,7 +4,7 @@
   <!-- Constants for robot dimensions -->
   <xacro:property name="mass" value="1" /> <!-- arbitrary value for mass -->
-  <xacro:property name="diameter" value="0.667" />
-  <xacro:property name="height1" value="0.1" /> <!-- base link -->
-  <xacro:property name="height2" value="0.35" /> <!-- link 1 -->
+  <xacro:property name="diameter" value="0.0667" />
+  <xacro:property name="height1" value="0.01" /> <!-- base link -->
+  <xacro:property name="height2" value="0.035" /> <!-- link 1 -->
   <joint name="${prefix}base_joint" type="fixed">
     <xacro:insert_block name="origin" />
@@ -69,5 +69,5 @@
   </link>
   <joint name="${prefix}marker_joint" type="fixed">
-    <origin xyz="${diameter/2-0.05} 0 ${height2+0.05/2}" rpy="0 0 0" />
+    <origin xyz="${0.3/2} 0 ${height2+0.01}" rpy="0 0 0" />
     <parent link="${prefix}link1"/>
     <child link="${prefix}marker_link" />
@@ -78,7 +78,7 @@
       <origin xyz="0 0 0" rpy="0 0 0"/>
       <geometry>
-        <cylinder radius="0.05" length="0.05"/>
+        <box size="0.3 0.02 0.02"/>
       </geometry>
-      <material name="orange"/>
+      <material name="blue"/>
     </visual>
   </link>
