Commit message: change name

File: rm_motors_example/urdf/rm_motors_description.urdf.xacro (robot description, xacro)
@@ -1,5 +1,5 @@
 <?xml version="1.0"?>
 <robot xmlns:xacro="http://www.ros.org/wiki/xacro">
-  <xacro:macro name="gm6020" params="parent prefix *origin">
+  <xacro:macro name="rm_motors" params="parent prefix *origin">
   <!-- Constants for robot dimensions -->
   <xacro:property name="mass" value="1" /> <!-- arbitrary value for mass -->

Commit message: minor fixes

File: rm_motors_example/urdf/rm_motors_description.urdf.xacro (robot description, xacro)
@@ -42,5 +42,5 @@
     <axis xyz="0 0 1"/>
     <dynamics damping="0.7"/>
-    <limit effort="100" velocity="1.0"/>
+    <limit effort="100" velocity="10.0"/>
   </joint>
   <!-- Middle Link -->
